File: 16_STEP_DOWN.kicad_pcb (KiCad board)
At the start: 2 copper layers, 20.3 x 20.3 mm, 12 parts, among them J1 Conn_01x01, J2 Conn_01x01, J3 Conn_01x01, J4 Conn_01x01, J5 Conn_01x01

Commit message: prêt pour fabrication
ajout sct2325
routage
Parts:
- removed H1, H2, H3, H4, H5, H6: percage, Chimere:trou
- added C1: 100nF, Capacitor_SMD:C_0603_1608Metric, F.Cu at (114.6, 74.2)
- added C2: 10uF/50V, Capacitor_SMD:C_1210_3225Metric, F.Cu at (115.6, 71.7)
- added C3: 100nF, Capacitor_SMD:C_0603_1608Metric, F.Cu at (109.1, 67.2)
- added C5: 10uF/50V, Capacitor_SMD:C_1210_3225Metric, F.Cu at (109.2, 77.7)
- added D1: 1N5819W, Diode_SMD:D_SOD-123F, F.Cu at (110.9, 63.5)
- added D2: LED_ALT, Diode_SMD:D_0603_1608Metric, F.Cu at (112.1, 76.7)
- added L1: MWSA0402S-100MT, Chimere:L_Sunlord_MWSA0402S_4.2x4.4x2.0mm, F.Cu at (106.1, 71.7)
- added R1: 10k, Resistor_SMD:R_0603_1608Metric, F.Cu at (114.1, 76.7)
- added U1: SCT2325, Package_TO_SOT_SMD:TSOT-23-6_HandSoldering, F.Cu at (110.6, 71.2)
- moved C4 24.5 mm to (106.7, 77.5), turned to 270 degrees
- moved J5 5.08 mm to (116.8, 63.5)
- moved J1 2.54 mm to (104.1, 66.0)
- moved J2 2.54 mm to (104.1, 63.5)
- moved J3 2.54 mm to (104.1, 76.2)
- moved J4 2.54 mm to (104.1, 78.7)
- renumbered C1 to C4
Connections:
- J4 pad 1: ENABLE -> EN
Routing:
- net GND: track 0.00 -> 75.5 mm, vias 0 -> 22
- net V_BRUT_P: track 0.00 -> 17.9 mm
- net 5V: track 0.00 -> 15.6 mm
- net Net-(C3-Pad2): track 0.00 -> 12.6 mm
- net EN: track 0.00 -> 11.1 mm, vias 0 -> 1
- net V_BRUT: track 0.00 -> 5.35 mm
- net Net-(D2-Pad1): track 0.00 -> 4.01 mm
- net Net-(C3-Pad1): track 0.00 -> 3.37 mm
- added copper zone on F.Cu, net 5V
- added copper zone on F.Cu, net Net-(C3-Pad2)
- added copper zone on F.Cu, net V_BRUT
- added copper zone on F.Cu, net V_BRUT_P
Other:
- outline, holes or cut-outs redrawn
- board text added: "EN"
- board text added: "VIN"

Commit message: maj split librairies
Parts:
- J1, J2, J3, J4, J5: footprint Chimere:Castellated_conn -> Chimere_mods:Castellated_conn
- L1: footprint Chimere:L_Sunlord_MWSA0402S_4.2x4.4x2.0mm -> Chimere_comps:L_Sunlord_MWSA0402S_4.2x4.4x2.0mm
