File: 16_STEP_DOWN.sch (KiCad schematic (older format))
At the start: 20 parts, among them J1 Conn_01x01, J2 Conn_01x01, J3 Conn_01x01, J4 Conn_01x01, J5 Conn_01x01

Commit message: prêt pour fabrication
ajout sct2325
routage
Parts:
- removed H1, H2, H3, H4, H5, H6: percage, Chimere:trou, symbol Mechanical:MountingHole
- added U1: SCT2325, Package_TO_SOT_SMD:TSOT-23-6_HandSoldering, symbol Chimere:SCT2325
- gave numbers to parts that had none: 9
Connections:
- net 5V: now also L1.1, U1.1 (VS)
- net GND: now also U1.4 (GND)
- net V_BRUT_P: now also U1.3 (VIN)
- net at C3.1: now also U1.6 (BST)
- net at C3.2: now also L1.2, U1.5 (SW)
- net ENABLE renamed EN
- net EN: now also U1.2 (EN)
Other:
- moved on the sheet: C3, C4, C5, D2, L1, R1
Changed lines of the file:
@@
 Wire Wire Line
 	1525 7250 1600 7250
-$Comp
-L Mechanical:MountingHole H1
-U 1 1 607A1C81
-P 4475 6950
-F 0 "H1" H 4575 6996 50  0000 L CNN
-F 1 "percage" H 4575 6905 50  0000 L CNN
-F 2 "Chimere:trou" H 4475 6950 50  0001 C CNN
-F 3 "~" H 4475 6950 50  0001 C CNN
-	1    4475 6950
-	1    0    0    -1
-$EndComp
-$Comp
-L Mechanical:MountingHole H5
-U 1 1 607A3404
-P 4475 7225
-F 0 "H5" H 4575 7271 50  0000 L CNN
-F 1 "percage" H 4575 7180 50  0000 L CNN
-F 2 "Chimere:trou" H 4475 7225 50  0001 C CNN
-F 3 "~" H 4475 7225 50  0001 C CNN
-	1    4475 7225
-	1    0    0    -1
-$EndComp
-$Comp
-L Mechanical:MountingHole H2
-U 1 1 607A3C27
-P 5025 6950
-F 0 "H2" H 5125 6996 50  0000 L CNN
-F 1 "percage" H 5125 6905 50  0000 L CNN
-F 2 "Chimere:trou" H 5025 6950 50  0001 C CNN
-F 3 "~" H 5025 6950 50  0001 C CNN
-	1    5025 6950
-	1    0    0    -1
-$EndComp
-$Comp
-L Mechanical:MountingHole H6
-U 1 1 607A3C2D
-P 5025 7225
-F 0 "H6" H 5125 7271 50  0000 L CNN
-F 1 "percage" H 5125 7180 50  0000 L CNN
-F 2 "Chimere:trou" H 5025 7225 50  0001 C CNN
-F 3 "~" H 5025 7225 50  0001 C CNN
-	1    5025 7225
-	1    0    0    -1
-$EndComp
-$Comp
-L Mechanical:MountingHole H3
-U 1 1 607A502A
-P 5500 6950
-F 0 "H3" H 5600 6996 50  0000 L CNN
-F 1 "percage" H 5600 6905 50  0000 L CNN
-F 2 "Chimere:trou" H 5500 6950 50  0001 C CNN
-F 3 "~" H 5500 6950 50  0001 C CNN
-	1    5500 6950
-	1    0    0    -1
-$EndComp
-$Comp
-L Mechanical:MountingHole H4
-U 1 1 607A5036
-P 6050 6950
-F 0 "H4" H 6150 6996 50  0000 L CNN
-F 1 "percage" H 6150 6905 50  0000 L CNN
-F 2 "Chimere:trou" H 6050 6950 50  0001 C CNN
-F 3 "~" H 6050 6950 50  0001 C CNN
-	1    6050 6950
-	1    0    0    -1
-$EndComp
 Text GLabel 1525 6725 0    50   Input ~ 0
 GND
@@
 5V
 $Comp
-L Device:C C?
+L Device:C C4
 U 1 1 60AF6DD6
-P 8100 3175
-F 0 "C?" H 8215 3221 50  0000 L CNN
-F 1 "100nF" H 8215 3130 50  0000 L CNN
-F 2 "Capacitor_SMD:C_0603_1608Metric" H 8138 3025 50  0001 C CNN
-F 3 "C14663" H 8100 3175 50  0001 C CNN
-	1    8100 3175
+P 4650 2950
+F 0 "C4" H 4765 2996 50  0000 L CNN
+F 1 "100nF" H 4765 2905 50  0000 L CNN
+F 2 "Capacitor_SMD:C_0603_1608Metric" H 4688 2800 50  0001 C CNN
+F 3 "C14663" H 4650 2950 50  0001 C CNN
+	1    4650 2950
 	1    0    0    -1
 $EndComp
-Text GLabel 8050 3025 0    50   Input ~ 0
+Text GLabel 4600 2800 0    50   Input ~ 0
 5V
-Text GLabel 8050 3325 0    50   Input ~ 0
+Text GLabel 4600 3100 0    50   Input ~ 0
 GND
 Wire Wire Line
-	8050 3025 8100 3025
-Wire Wire Line
-	8050 3325 8100 3325
+	4600 2800 4650 2800
+Wire Wire Line
+	4600 3100 4650 3100
 Wire Wire Line
 	2875 6750 2950 6750
@@
 V_BRUT
 Text GLabel 1525 7250 0    50   Input ~ 0
-ENABLE
+EN
 $Bitmap
 Pos 1550 1450
@@
 inductance:\nMWSA0402S-100MT\nC408339\nSMD-4.2*4.4*2.0
 $Comp
-L Device:C C?
+L Device:C C5
 U 1 1 60B0B3C0
-P 8725 3175
-F 0 "C?" H 8840 3221 50  0000 L CNN
-F 1 "10uF/50V" H 8840 3130 50  0000 L CNN
-F 2 "Capacitor_SMD:C_1210_3225Metric" H 8763 3025 50  0001 C CNN
-F 3 "C337485" H 8725 3175 50  0001 C CNN
-	1    8725 3175
+P 5275 2950
+F 0 "C5" H 5390 2996 50  0000 L CNN
+F 1 "10uF/50V" H 5390 2905 50  0000 L CNN
+F 2 "Capacitor_SMD:C_1210_3225Metric" H 5313 2800 50  0001 C CNN
+F 3 "C337485" H 5275 2950 50  0001 C CNN
+	1    5275 2950
 	1    0    0    -1
 $EndComp
-Text GLabel 8675 3025 0    50   Input ~ 0
+Text GLabel 5225 2800 0    50   Input ~ 0
 5V
-Text GLabel 8675 3325 0    50   Input ~ 0
+Text GLabel 5225 3100 0    50   Input ~ 0
 GND
 Wire Wire Line
-	8675 3025 8725 3025
-Wire Wire Line
-	8675 3325 8725 3325
+	5225 2800 5275 2800
+Wire Wire Line
+	5225 3100 5275 3100
 $Comp
-L Device:C C?
+L Device:C C1
 U 1 1 60B0BFEF
 P 5725 775
-F 0 "C?" H 5840 821 50  0000 L CNN
+F 0 "C1" H 5840 821 50  0000 L CNN
 F 1 "100nF" H 5840 730 50  0000 L CNN
 F 2 "Capacitor_SMD:C_0603_1608Metric" H 5763 625 50  0001 C CNN
@@
 	5675 925  5725 925
 $Comp
-L Device:C C?
+L Device:C C2
 U 1 1 60B0BFF9
 P 6425 775
-F 0 "C?" H 6540 821 50  0000 L CNN
+F 0 "C2" H 6540 821 50  0000 L CNN
 F 1 "10uF/50V" H 6540 730 50  0000 L CNN
 F 2 "Capacitor_SMD:C_1210_3225Metric" H 6463 625 50  0001 C CNN
@@
 V_BRUT_P
 $Comp
-L Device:C C?
+L Device:C C3
 U 1 1 60B0EA9D
-P 5400 2025
-F 0 "C?" H 5515 2071 50  0000 L CNN
-F 1 "100nF" H 5515 1980 50  0000 L CNN
-F 2 "Capacitor_SMD:C_0603_1608Metric" H 5438 1875 50  0001 C CNN
-F 3 "C14663" H 5400 2025 50  0001 C CNN
-	1    5400 2025
-	1    0    0    -1
+P 5475 1650
+F 0 "C3" H 5590 1696 50  0000 L CNN
+F 1 "100nF" H 5590 1605 50  0000 L CNN
+F 2 "Capacitor_SMD:C_0603_1608Metric" H 5513 1500 50  0001 C CNN
+F 3 "C14663" H 5475 1650 50  0001 C CNN
+	1    5475 1650
+	0    -1   -1   0
 $EndComp
 $Comp
-L Device:D_ALT D?
+L Device:D_ALT D1
 U 1 1 60B0F6BE
 P 4550 775
-F 0 "D?" H 4550 558 50  0000 C CNN
+F 0 "D1" H 4550 558 50  0000 C CNN
 F 1 "1N5819W" H 4550 649 50  0000 C CNN
 F 2 "Diode_SMD:D_SOD-123F" H 4550 775 50  0001 C CNN
@@
 Wire Wire Line
 	4700 775  4750 775
-Text GLabel 9450 2900 0    50   Input ~ 0
+Text GLabel 6000 2675 0    50   Input ~ 0
 5V
-Text GLabel 9425 3550 0    50   Input ~ 0
+Text GLabel 5975 3325 0    50   Input ~ 0
 GND
 $Comp
-L Device:LED_ALT D?
+L Device:LED_ALT D2
 U 1 1 60B1373B
-P 9500 3050
-F 0 "D?" V 9539 2932 50  0000 R CNN
-F 1 "LED_ALT" V 9448 2932 50  0000 R CNN
-F 2 "Diode_SMD:D_0603_1608Metric" H 9500 3050 50  0001 C CNN
-F 3 "C2286" H 9500 3050 50  0001 C CNN
-	1    9500 3050
+P 6050 2825
+F 0 "D2" V 6089 2707 50  0000 R CNN
+F 1 "LED_ALT" V 5998 2707 50  0000 R CNN
+F 2 "Diode_SMD:D_0603_1608Metric" H 6050 2825 50  0001 C CNN
+F 3 "C2286" H 6050 2825 50  0001 C CNN
+	1    6050 2825
 	0    -1   -1   0
 $EndComp
 $Comp
-L Device:R R?
+L Device:R R1
 U 1 1 60B1434A
-P 9500 3400
-F 0 "R?" H 9570 3446 50  0000 L CNN
-F 1 "10k" H 9570 3355 50  0000 L CNN
-F 2 "Resistor_SMD:R_0603_1608Metric" V 9430 3400 50  0001 C CNN
-F 3 "C25804" H 9500 3400 50  0001 C CNN
-	1    9500 3400
+P 6050 3175
+F 0 "R1" H 6120 3221 50  0000 L CNN
+F 1 "10k" H 6120 3130 50  0000 L CNN
+F 2 "Resistor_SMD:R_0603_1608Metric" V 5980 3175 50  0001 C CNN
+F 3 "C25804" H 6050 3175 50  0001 C CNN
+	1    6050 3175
 	1    0    0    -1
 $EndComp
 Wire Wire Line
-	9450 2900 9500 2900
-Wire Wire Line
-	9425 3550 9500 3550
-Wire Wire Line
-	9500 3200 9500 3250
+	6000 2675 6050 2675
+Wire Wire Line
+	5975 3325 6050 3325
+Wire Wire Line
+	6050 2975 6050 3025
 $Comp
-L Device:L L?
+L Device:L L1
 U 1 1 60B193A9
-P 5975 2350
-F 0 "L?" V 5794 2350 50  0000 C CNN
-F 1 "MWSA0402S-100MT" V 5885 2350 50  0000 C CNN
-F 2 "Chimere:L_Sunlord_MWSA0402S_4.2x4.4x2.0mm" H 5975 2350 50  0001 C CNN
-F 3 "C408339" H 5975 2350 50  0001 C CNN
-	1    5975 2350
+P 5850 1900
+F 0 "L1" V 5669 1900 50  0000 C CNN
+F 1 "MWSA0402S-100MT" V 5760 1900 50  0000 C CNN
+F 2 "Chimere:L_Sunlord_MWSA0402S_4.2x4.4x2.0mm" H 5850 1900 50  0001 C CNN
+F 3 "C408339" H 5850 1900 50  0001 C CNN
+	1    5850 1900
 	0    1    1    0
 $EndComp
-Text GLabel 4550 2400 0    50   Input ~ 0
+Text GLabel 4650 2000 0    50   Input ~ 0
 V_BRUT_P
-Text GLabel 6250 2350 2    50   Input ~ 0
+Text GLabel 6050 1900 2    50   Input ~ 0
 5V
+$Comp
+L Chimere:SCT2325 U1
+U 1 1 60B10DAA
+P 5025 1900
+F 0 "U1" H 5025 2225 50  0000 C CNN
+F 1 "SCT2325" H 5025 2134 50  0000 C CNN
+F 2 "Package_TO_SOT_SMD:TSOT-23-6_HandSoldering" H 5025 1900 50  0001 C CNN
+F 3 "C509064" H 5025 1900 50  0001 C CNN
+	1    5025 1900
+	1    0    0    -1
+$EndComp
+Wire Wire Line
+	4650 2000 4725 2000
+Text GLabel 5375 2000 2    50   Input ~ 0
+GND
+Wire Wire Line
+	5325 2000 5375 2000
+Wire Wire Line
+	5325 1800 5325 1650
+Wire Wire Line
+	5325 1900 5625 1900
+Wire Wire Line
+	5625 1900 5625 1650
+Wire Wire Line
+	5700 1900 5625 1900
+Connection ~ 5625 1900
+Wire Wire Line
+	6000 1900 6025 1900
+Wire Wire Line
+	4725 1800 4725 1250
+Wire Wire Line
+	4725 1250 6025 1250
+Wire Wire Line
+	6025 1250 6025 1900
+Connection ~ 6025 1900
+Wire Wire Line
+	6025 1900 6050 1900
+Text GLabel 4650 1900 0    50   Input ~ 0
+EN
+Wire Wire Line
+	4650 1900 4725 1900
 $EndSCHEMATC

Commit message: maj split librairies
Parts:
- J1, J2, J3, J4, J5: footprint Chimere:Castellated_conn -> Chimere_mods:Castellated_conn
- L1: footprint Chimere:L_Sunlord_MWSA0402S_4.2x4.4x2.0mm -> Chimere_comps:L_Sunlord_MWSA0402S_4.2x4.4x2.0mm
- U1: symbol Chimere:SCT2325 -> Chimere_comps:SCT2325
Changed lines of the file:
@@
 F 0 "J1" H 1880 6767 50  0000 L CNN
 F 1 "Conn_01x01" H 1880 6676 50  0000 L CNN
-F 2 "Chimere:Castellated_conn" H 1800 6725 50  0001 C CNN
+F 2 "Chimere_mods:Castellated_conn" H 1800 6725 50  0001 C CNN
 F 3 "~" H 1800 6725 50  0001 C CNN
 	1    1800 6725
@@
 F 0 "J3" H 1880 7117 50  0000 L CNN
 F 1 "Conn_01x01" H 1880 7026 50  0000 L CNN
-F 2 "Chimere:Castellated_conn" H 1800 7075 50  0001 C CNN
+F 2 "Chimere_mods:Castellated_conn" H 1800 7075 50  0001 C CNN
 F 3 "~" H 1800 7075 50  0001 C CNN
 	1    1800 7075
@@
 F 0 "J2" H 1880 6942 50  0000 L CNN
 F 1 "Conn_01x01" H 1880 6851 50  0000 L CNN
-F 2 "Chimere:Castellated_conn" H 1800 6900 50  0001 C CNN
+F 2 "Chimere_mods:Castellated_conn" H 1800 6900 50  0001 C CNN
 F 3 "~" H 1800 6900 50  0001 C CNN
 	1    1800 6900
@@
 F 0 "J5" H 3230 6792 50  0000 L CNN
 F 1 "Conn_01x01" H 3230 6701 50  0000 L CNN
-F 2 "Chimere:Castellated_conn" H 3150 6750 50  0001 C CNN
+F 2 "Chimere_mods:Castellated_conn" H 3150 6750 50  0001 C CNN
 F 3 "~" H 3150 6750 50  0001 C CNN
 	1    3150 6750
@@
 F 0 "J4" H 1880 7292 50  0000 L CNN
 F 1 "Conn_01x01" H 1880 7201 50  0000 L CNN
-F 2 "Chimere:Castellated_conn" H 1800 7250 50  0001 C CNN
+F 2 "Chimere_mods:Castellated_conn" H 1800 7250 50  0001 C CNN
 F 3 "~" H 1800 7250 50  0001 C CNN
 	1    1800 7250
@@
 F 0 "L1" V 5669 1900 50  0000 C CNN
 F 1 "MWSA0402S-100MT" V 5760 1900 50  0000 C CNN
-F 2 "Chimere:L_Sunlord_MWSA0402S_4.2x4.4x2.0mm" H 5850 1900 50  0001 C CNN
+F 2 "Chimere_comps:L_Sunlord_MWSA0402S_4.2x4.4x2.0mm" H 5850 1900 50  0001 C CNN
 F 3 "C408339" H 5850 1900 50  0001 C CNN
 	1    5850 1900
@@
 5V
 $Comp
-L Chimere:SCT2325 U1
+L Chimere_comps:SCT2325 U1
 U 1 1 60B10DAA
 P 5025 1900
